File: Thermometry_Enclosure/I2C_Bus.kicad_sch (KiCad schematic)
At the start: 13 parts, among them J62 JST_SH_Conn_01x04, J63 JST_SH_Conn_01x04, J64 JST_SH_Conn_01x04, J65 JST_SH_Conn_01x04, J66 JST_SH_Conn_01x04

Commit message: update
Parts:
- removed R3, R4, R5, R6, R7, R8: 4.7K, Resistor_SMD:R_0603_1608Metric_Pad0.98x0.95mm_HandSolder, symbol Device:R
