File: Thermometry_Enclosure/HDMI_ports.kicad_sch (KiCad schematic)
At the start: 40 parts, among them J1 HDMI_A_1.4, J16 JST_SH_Conn_01x04_D HEad, J17 JST_SH_Conn_01x04_3Head B, J18 JST_SH_Conn_01x04_3Head A, J19 JST_SH_Conn_01x04_4Head B, J2 HDMI_A_1.4, J20 JST_SH_Conn_01x04_Still, J21 JST_SH_Conn_01x04_4Head A, J22 JST_SH_Conn_01x04_4Pump Diode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, J23 JST_SH_Conn_01x04_4Pump Diode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, J24 JST_SH_Conn_01x04_3Pump Diode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, J25 JST_SH_Conn_01x04_3Pump Diode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, J26 JST_SH_Conn_01x04_4Switch Dio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, J27 JST_SH_Conn_01x04_Condenser, J28 JST_SH_Conn_01x04_4Switch Dio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, J29 JST_SH_Conn_01x04_3Switch Dio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, J3 HDMI_A_1.4, J30 Conn_01x02_Still Heater, J31 JST_SH_Conn_01x04_3Switch Dio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, J32 Conn_01x02_15 pin Extra, J33 Conn_01x02_4SwitchHeater B, J34 Conn_01x02_4SwitchHeater A, J35 Conn_01x02_3SwitchHeater B, J36 Conn_01x02_3SwitchHeater A, J37 JST_SH_Conn_01x04_40K Diode, J38 Conn_01x02_4PumpHeater B, J39 Conn_01x02_4PumpHeater A, J4 HDMI_A_1.4, J40 Conn_01x02_3PumpHeater B, J41 Conn_01x02_3PumpHeater A, J42 JST_SH_Conn_01x04_4K Diode, J43 Conn_01x02_Extra B, J44 Conn_01x02_Extra A, J45 Conn_01x02_Extra B, J46 Conn_01x02_Extra A, J5 HDMI_A_1.4, J6 HDMI_A_1.4, J7 HDMI_A_1.4, J8 HDMI_A_1.4, J9 HDMI_A_1.4

Commit message: Removed files unrelated
Parts:
- J1, J2, J3, J4, J5, J6, J7, J8, J9: footprint 0Library:HDMI-TH_HDMI-019A -> 0Library:HDMI-TH_HYC12-HDMIA19-61; LCSC C369072 -> C711354
Changed lines of the file:
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@@
     (property "Reference" "J3" (id 0) (at 173.355 14.0802 90))
     (property "Value" "HDMI_A_1.4" (id 1) (at 173.355 16.6171 90))
-    (property "Footprint" "0Library:HDMI-TH_HDMI-019A" (id 2) (at 173.355 27.305 0)
+    (property "Footprint" "0Library:HDMI-TH_HYC12-HDMIA19-61" (id 2) (at 173.355 27.305 0)
       (effects (font (size 1.27 1.27)) hide)
     )
@@
       (effects (font (size 1.27 1.27)) hide)
     )
-    (property "LCSC" "C369072" (id 4) (at 173.355 27.94 0)
+    (property "LCSC" "C711354" (id 4) (at 173.355 27.94 0)
       (effects (font (size 1.27 1.27)) hide)
     )
@@
     (property "Reference" "J6" (id 0) (at 170.18 101.0752 90))
     (property "Value" "HDMI_A_1.4" (id 1) (at 170.18 103.6121 90))
-    (property "Footprint" "0Library:HDMI-TH_HDMI-019A" (id 2) (at 170.18 114.3 0)
+    (property "Footprint" "0Library:HDMI-TH_HYC12-HDMIA19-61" (id 2) (at 170.18 114.3 0)
       (effects (font (size 1.27 1.27)) hide)
     )
@@
       (effects (font (size 1.27 1.27)) hide)
     )
-    (property "LCSC" "C369072" (id 4) (at 170.18 114.935 0)
+    (property "LCSC" "C711354" (id 4) (at 170.18 114.935 0)
       (effects (font (size 1.27 1.27)) hide)
     )
@@
     (property "Reference" "J1" (id 0) (at 43.815 14.0802 90))
     (property "Value" "HDMI_A_1.4" (id 1) (at 43.815 16.6171 90))
-    (property "Footprint" "0Library:HDMI-TH_HDMI-019A" (id 2) (at 43.815 27.305 0)
+    (property "Footprint" "0Library:HDMI-TH_HYC12-HDMIA19-61" (id 2) (at 43.815 27.305 0)
       (effects (font (size 1.27 1.27)) hide)
     )
@@
       (effects (font (size 1.27 1.27)) hide)
     )
-    (property "LCSC" "C369072" (id 4) (at 43.815 27.94 0)
+    (property "LCSC" "C711354" (id 4) (at 43.815 27.94 0)
       (effects (font (size 1.27 1.27)) hide)
     )
@@
     (property "Reference" "J8" (id 0) (at 105.41 222.3602 90))
     (property "Value" "HDMI_A_1.4" (id 1) (at 105.41 224.8971 90))
-    (property "Footprint" "0Library:HDMI-TH_HDMI-019A" (id 2) (at 105.41 235.585 0)
+    (property "Footprint" "0Library:HDMI-TH_HYC12-HDMIA19-61" (id 2) (at 105.41 235.585 0)
       (effects (font (size 1.27 1.27)) hide)
     )
@@
       (effects (font (size 1.27 1.27)) hide)
     )
-    (property "LCSC" "C369072" (id 4) (at 105.41 236.22 0)
+    (property "LCSC" "C711354" (id 4) (at 105.41 236.22 0)
       (effects (font (size 1.27 1.27)) hide)
     )
@@
     (property "Reference" "J2" (id 0) (at 109.22 14.0802 90))
     (property "Value" "HDMI_A_1.4" (id 1) (at 109.22 16.6171 90))
-    (property "Footprint" "0Library:HDMI-TH_HDMI-019A" (id 2) (at 109.22 27.305 0)
+    (property "Footprint" "0Library:HDMI-TH_HYC12-HDMIA19-61" (id 2) (at 109.22 27.305 0)
       (effects (font (size 1.27 1.27)) hide)
     )
@@
       (effects (font (size 1.27 1.27)) hide)
     )
-    (property "LCSC" "C369072" (id 4) (at 109.22 27.94 0)
+    (property "LCSC" "C711354" (id 4) (at 109.22 27.94 0)
       (effects (font (size 1.27 1.27)) hide)
     )
@@
     (property "Reference" "J4" (id 0) (at 40.64 101.0752 90))
     (property "Value" "HDMI_A_1.4" (id 1) (at 40.64 103.6121 90))
-    (property "Footprint" "0Library:HDMI-TH_HDMI-019A" (id 2) (at 40.64 114.3 0)
+    (property "Footprint" "0Library:HDMI-TH_HYC12-HDMIA19-61" (id 2) (at 40.64 114.3 0)
       (effects (font (size 1.27 1.27)) hide)
     )
@@
       (effects (font (size 1.27 1.27)) hide)
     )
-    (property "LCSC" "C369072" (id 4) (at 40.64 114.935 0)
+    (property "LCSC" "C711354" (id 4) (at 40.64 114.935 0)
       (effects (font (size 1.27 1.27)) hide)
     )
@@
       (effects (font (size 1.27 1.27)) (justify left))
     )
-    (property "Footprint" "0Library:HDMI-TH_HDMI-019A" (id 2) (at 44.45 235.585 0)
+    (property "Footprint" "0Library:HDMI-TH_HYC12-HDMIA19-61" (id 2) (at 44.45 235.585 0)
       (effects (font (size 1.27 1.27)) hide)
     )
@@
       (effects (font (size 1.27 1.27)) hide)
     )
-    (property "LCSC" "C369072" (id 4) (at 44.45 236.22 0)
+    (property "LCSC" "C711354" (id 4) (at 44.45 236.22 0)
       (effects (font (size 1.27 1.27)) hide)
     )
@@
       (effects (font (size 1.27 1.27)) (justify left))
     )
-    (property "Footprint" "0Library:HDMI-TH_HDMI-019A" (id 2) (at 166.37 235.585 0)
+    (property "Footprint" "0Library:HDMI-TH_HYC12-HDMIA19-61" (id 2) (at 166.37 235.585 0)
       (effects (font (size 1.27 1.27)) hide)
     )
@@
       (effects (font (size 1.27 1.27)) hide)
     )
-    (property "LCSC" "C369072" (id 4) (at 166.37 236.22 0)
+    (property "LCSC" "C711354" (id 4) (at 166.37 236.22 0)
       (effects (font (size 1.27 1.27)) hide)
     )
@@
     (property "Reference" "J5" (id 0) (at 106.045 101.0752 90))
     (property "Value" "HDMI_A_1.4" (id 1) (at 106.045 103.6121 90))
-    (property "Footprint" "0Library:HDMI-TH_HDMI-019A" (id 2) (at 106.045 114.3 0)
+    (property "Footprint" "0Library:HDMI-TH_HYC12-HDMIA19-61" (id 2) (at 106.045 114.3 0)
       (effects (font (size 1.27 1.27)) hide)
     )
@@
       (effects (font (size 1.27 1.27)) hide)
     )
-    (property "LCSC" "C369072" (id 4) (at 106.045 114.935 0)
-      (effects (font (size 1.27 1.27)) hide)
-    )
+    (property "LCSC" "C711354" (id 4) (at 106.045 114.935 0)
+      (effects (font (size 1.27 1.27)) hide)
+    )
