File: Thermometry_Enclosure/Thermometry_Enclosure.kicad_pcb (KiCad board)
At the start: 2 copper layers, 102 parts, among them J1 HDMI_A_1.4, J10 JST_SH_Conn_01x04_UART 1, J11 JST_SH_Conn_01x04_MUX 1, J12 JST_SH_Conn_01x04_UART 0, J13 JST_SH_Conn_01x04_MUX 0, J14 Conn_01x07_Female, J15 Conn_01x07_Female, J16 JST_SH_Conn_01x04_D HEad, J17 JST_SH_Conn_01x04_3Head B, J18 JST_SH_Conn_01x04_3Head A, J19 JST_SH_Conn_01x04_4Head B, J2 HDMI_A_1.4, J20 JST_SH_Conn_01x04_Still, J21 JST_SH_Conn_01x04_4Head A, J22 JST_SH_Conn_01x04_4Pump Diode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, J23 JST_SH_Conn_01x04_4Pump Diode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, J24 JST_SH_Conn_01x04_3Pump Diode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, J25 JST_SH_Conn_01x04_3Pump Diode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, J26 JST_SH_Conn_01x04_4Switch Dio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, J27 JST_SH_Conn_01x04_Condenser, J28 JST_SH_Conn_01x04_4Switch Dio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, J29 JST_SH_Conn_01x04_3Switch Dio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, J3 HDMI_A_1.4, J30 Conn_01x02_Still Heater, J31 JST_SH_Conn_01x04_3Switch Dio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, J32 Conn_01x02_15 pin Extra, J33 Conn_01x02_4SwitchHeater B, J34 Conn_01x02_4SwitchHeater A, J35 Conn_01x02_3SwitchHeater B, J36 Conn_01x02_3SwitchHeater A, J37 JST_SH_Conn_01x04_40K Diode, J38 Conn_01x02_4PumpHeater B, J39 Conn_01x02_4PumpHeater A, J4 HDMI_A_1.4, J40 Conn_01x02_3PumpHeater B, J41 Conn_01x02_3PumpHeater A, J42 JST_SH_Conn_01x04_4K Diode, J43 Conn_01x02_Extra B, J44 Conn_01x02_Extra A, J45 Conn_01x02_Extra B, J46 Conn_01x02_Extra A, J47 Conn_01x02_Lockin 5V, J48 Conn_01x03, J49 JST_SH_Conn_01x04_4K Diode, J5 HDMI_A_1.4, J50 Conn_01x02_Female_HP1, J51 Conn_01x02_Female_HP2, J52 Conn_01x02_Female_HP3, J53 Conn_01x04, J54 JST_SH_Conn_01x04_40K Diode, J55 Conn_01x07_Female, J56 Conn_01x05_Female_LPH, J57 Conn_01x07_Female, J58 Conn_01x07_Female, J59 Conn_01x07_Female, J6 HDMI_A_1.4, J60 Conn_01x02_Female_HP4, J61 Conn_01x03, J62 JST_SH_Conn_01x04, J63 JST_SH_Conn_01x04, J64 JST_SH_Conn_01x04, J65 JST_SH_Conn_01x04, J66 JST_SH_Conn_01x04, J7 HDMI_A_1.4, J8 HDMI_A_1.4, J9 HDMI_A_1.4

Commit message: update
Parts:
- removed R3, R4, R5, R6, R7, R8: 4.7K, Resistor_SMD:R_0603_1608Metric_Pad0.98x0.95mm_HandSolder
- added DC1: DC-044K-D025, 0Library:DC-IN-TH_DC-044K-D025, F.Cu at (1.00, -0.60)
- added H26: MountingHole, MountingHole:MountingHole_2.2mm_M2_Pad, F.Cu at (316.5, 58.4)
- added H27: MountingHole, MountingHole:MountingHole_2.2mm_M2_Pad, F.Cu at (329.5, 58.4)
- added H28: MountingHole, MountingHole:MountingHole_2.2mm_M2_Pad, F.Cu at (316.5, 91.4)
- added H29: MountingHole, MountingHole:MountingHole_2.2mm_M2_Pad, F.Cu at (329.5, 91.4)
- added H30: MountingHole_Pad, MountingHole:MountingHole_5.3mm_M5_Pad, F.Cu at (280.6, 106.0)
- added H31: MountingHole_Pad, MountingHole:MountingHole_5.3mm_M5_Pad, F.Cu at (72.2, 279.0)
- added H32: MountingHole_Pad, MountingHole:MountingHole_5.3mm_M5_Pad, F.Cu at (176.3, 279.0)
- added H33: MountingHole_Pad, MountingHole:MountingHole_5.3mm_M5_Pad, F.Cu at (280.6, 279.0)
- added H34: MountingHole_Pad, MountingHole:MountingHole_5.3mm_M5_Pad, F.Cu at (350.0, 35.0)
- added H35: MountingHole_Pad, MountingHole:MountingHole_5.3mm_M5_Pad, F.Cu at (176.3, 106.0)
- added H36: MountingHole_Pad, MountingHole:MountingHole_5.3mm_M5_Pad, F.Cu at (350.0, 150.0)
- added H37: MountingHole_Pad, MountingHole:MountingHole_5.3mm_M5_Pad, F.Cu at (72.2, 106.0)
- added H38: MountingHole_Pad, MountingHole:MountingHole_5.3mm_M5_Pad, F.Cu at (25.0, 175.0)
- added H39: MountingHole_Pad, MountingHole:MountingHole_5.3mm_M5_Pad, F.Cu at (25.0, 35.0)
- added H40: MountingHole_Pad, MountingHole:MountingHole_5.3mm_M5_Pad, F.Cu at (216.0, 44.0)
- added H41: MountingHole_Pad, MountingHole:MountingHole_6.5mm_Pad, F.Cu at (307.0, 246.5)
- added H41: MountingHole_Pad, MountingHole:MountingHole_6.5mm_Pad, F.Cu at (176.2, 243.0)
- added J67: Conn_01x02_Lockin 5V, Connector_JST:JST_PH_B2B-PH-K_1x02_P2.00mm_Vertical, F.Cu at (81.0, 152.0)
- added J68: Conn_01x02_HP_5V, Connector_JST:JST_PH_B2B-PH-K_1x02_P2.00mm_Vertical, F.Cu at (243.9, 104.3)
- added USB1: TYPE-604-T3, 0Library:USB-C-TH_TYPE-604-T3, F.Cu at (72.0, 236.0)
- added USB2: U-USBAS04P-F000, 0Library:USB-A-TH_U-A-24DD-Y-2, F.Cu at (72.0, 249.5)
- J50, J51, J52, J60: footprint Connector_JST:JST_PH_B2B-PH-K_1x02_P2.00mm_Vertical -> Connector_PinSocket_2.54mm:PinSocket_1x02_P2.54mm_Vertical
- moved H5 250.5 mm to (8.53, 46.1), turned to 90 degrees
- moved H7 248.6 mm to (70.5, 46.1), turned to 90 degrees
- moved J25 239.5 mm to (261.4, 39.1)
- moved H19 237.9 mm to (325.5, 145.9), turned to -90 degrees
- moved H3 234.7 mm to (159.5, 46.1), turned to 90 degrees
- moved J53 234.3 mm to (316.0, 205.5), turned to 0 degrees
- moved J23 232.9 mm to (261.4, 30.6)
- moved J49 229.9 mm to (331.8, 102.6), turned to 180 degrees
- moved J58 229.1 mm to (308.0, 218.2), turned to 180 degrees
- moved J31 226.3 mm to (270.9, 39.1)
- moved H4 216.7 mm to (97.5, 46.1), turned to 90 degrees
- moved J36 214.3 mm to (223.0, 157.0)
- moved J28 213.6 mm to (270.9, 30.6)
- moved J34 208.5 mm to (223.0, 147.0)
- moved J59 200.7 mm to (292.8, 218.2), turned to 180 degrees
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Routing:
- net +5V: track 0.00 -> 699.7 mm
- net Net-(J1-Pad12): track 0.00 -> 281.0 mm
- net Net-(J1-Pad10): track 0.00 -> 278.5 mm
- net Net-(J2-Pad12): track 0.00 -> 259.0 mm, vias 0 -> 3
- net Net-(J2-Pad10): track 0.00 -> 258.9 mm, vias 0 -> 3
- net Net-(J2-Pad9): track 0.00 -> 256.5 mm, vias 0 -> 2
- net Net-(J1-Pad9): track 0.00 -> 254.7 mm
- net Net-(J2-Pad7): track 0.00 -> 254.3 mm, vias 0 -> 2
- net Net-(J1-Pad7): track 0.00 -> 254.0 mm
- net Net-(J2-Pad6): track 0.00 -> 245.4 mm, vias 0 -> 2
- net Net-(J2-Pad4): track 0.00 -> 240.5 mm, vias 0 -> 2
- net Net-(J2-Pad3): track 0.00 -> 235.9 mm, vias 0 -> 2
- net Net-(J2-Pad1): track 0.00 -> 235.3 mm, vias 0 -> 2
- net Net-(J30-Pad1): track 0.00 -> 189.8 mm
- net Net-(J30-Pad2): track 0.00 -> 188.6 mm
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- added copper zone on B.Cu, net GND
- added copper zone on F.Cu, net GND
Other:
- board outline added: 417 x 300.6 mm
- board text added: "2 x Diode Boards"
- board text added: "2xUART Mux Boards"
- board text added: "3Head A"
- board text added: "3Head B"
- board text added: "3Pump Diode A"
- board text added: "3Pump Diode B"
- board text added: "3Pump Heater A"
- board text added: "3Pump Heater B"
- board text added: "3Switch Diode A"
- board text added: "3Switch Diode B"
- board text added: "3switch Heater A"
- board text added: "3switch Heater B"
- board text added: "3x Lockin Boards"
- board text added: "4 x Diode Boards"
- board text added: "40K Diode"
- board text added: "4Head A"
- board text added: "4Head B"
- board text added: "4K Diode"
- board text added: "4Pump Diode A"
- board text added: "4Pump Diode B"
- board text added: "4Pump Heater A"
- board text added: "4Pump Heater B"
- board text added: "4Switch Diode A"
- board text added: "4Switch Diode B"
- board text added: "4switch Heater A"
- board text added: "4switch Heater B"
- board text added: "4x High Power Heater Boards"
- board text added: "4x Lockin Boards"
- board text added: "Condenser"
- board text added: "DHead"
- board text added: "Extra"
- board text added: "Extra A1"
- board text added: "Extra A2"
- board text added: "Extra B1"
- board text added: "Extra B2"
- board text added: "HP1 CTRL EN"
- board text added: "HP2 CTRL EN"
- board text added: "HP3 CTRL EN"
- board text added: "HP4 CTRL EN"
- board text added: "LPH LD CLK DI"
- board text added: "MUX 0"
- board text added: "MUX 1"
- board text added: "Still"
- board text added: "Still Heater"
- board text added: "UART 0"
- board text added: "UART 1"

Commit message: Removed files unrelated
Parts:
- J1, J2, J3, J4, J5, J6, J7, J8, J9: footprint 0Library:HDMI-TH_HDMI-019A -> 0Library:HDMI-TH_HYC12-HDMIA19-61
- moved J1 1.20 mm to (25.4, -1.20)
- moved J2 1.20 mm to (63.5, -1.20)
- moved J3 1.20 mm to (101.6, -1.20)
- moved J4 1.20 mm to (139.7, -1.20)
- moved J5 1.20 mm to (177.8, -1.20)
- moved J6 1.20 mm to (215.9, -1.20)
- moved J7 1.20 mm to (254.0, -1.20)
- moved J8 1.20 mm to (292.1, -1.20)
- moved J9 1.20 mm to (330.2, -1.20)
Routing:
- net GND: track 8.80 -> 66.4 mm, vias 3 -> 2
- net Net-(J40-Pad2): track 125.0 -> 119.9 mm
- net Net-(J1-Pad10): track 278.5 -> 275.0 mm
- net Net-(J3-Pad6): track 127.6 -> 124.2 mm
- net Net-(J35-Pad1): track 182.5 -> 185.8 mm
- net Net-(J32-Pad1): track 23.6 -> 26.7 mm
- net Net-(J2-Pad10): track 258.9 -> 262.0 mm
- net Net-(J42-Pad1): track 45.4 -> 48.5 mm
- net Net-(J40-Pad1): track 116.0 -> 119.0 mm
- net Net-(J1-Pad12): track 281.0 -> 278.0 mm
- net Net-(J24-Pad2): track 181.6 -> 184.5 mm
- net Net-(J1-Pad6): track 63.8 -> 66.7 mm
- net Net-(J35-Pad2): track 181.6 -> 184.4 mm
- net Net-(J45-Pad2): track 30.0 -> 27.3 mm
- net Net-(J29-Pad3): track 153.5 -> 156.2 mm
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