File: Thermometry_Enclosure/Thermometry_Enclosure.kicad_sch (KiCad schematic)
At the start: 49 parts, among them J10 JST_SH_Conn_01x04_UART 1, J11 JST_SH_Conn_01x04_MUX 1, J12 JST_SH_Conn_01x04_UART 0, J13 JST_SH_Conn_01x04_MUX 0, J14 Conn_01x07_Female, J15 Conn_01x07_Female, J47 Conn_01x02_Lockin 5V, J48 Conn_01x03, J49 JST_SH_Conn_01x04_4K Diode, J50 Conn_01x02_Female_HP1, J51 Conn_01x02_Female_HP2, J52 Conn_01x02_Female_HP3, J53 Conn_01x04, J54 JST_SH_Conn_01x04_40K Diode, J55 Conn_01x07_Female, J56 Conn_01x05_Female_LPH, J57 Conn_01x07_Female, J58 Conn_01x07_Female, J59 Conn_01x07_Female, J60 Conn_01x02_Female_HP4, J61 Conn_01x03

Commit message: update
Parts:
- added DC1: DC-044K-D025, 0Library:DC-IN-TH_DC-044K-D025, symbol 0Therm_Enclosure:DC-044K-D025
- added H26, H27, H28, H29: MountingHole, MountingHole:MountingHole_2.2mm_M2_Pad, symbol Mechanical:MountingHole
- added H30, H31, H32, H33, H34, H35, H36, H37, H38, H39, H40: MountingHole_Pad, MountingHole:MountingHole_5.3mm_M5_Pad, symbol Mechanical:MountingHole_Pad
- added H41: MountingHole_Pad, MountingHole:MountingHole_6.5mm_Pad, symbol Mechanical:MountingHole_Pad
- added J67: Conn_01x02_Lockin 5V, Connector_JST:JST_PH_B2B-PH-K_1x02_P2.00mm_Vertical, symbol Connector_Generic:Conn_01x02
- added J68: Conn_01x02_HP_5V, Connector_JST:JST_PH_B2B-PH-K_1x02_P2.00mm_Vertical, symbol Connector_Generic:Conn_01x02
- added USB1: TYPE-604-T3, 0Library:USB-C-TH_TYPE-604-T3, symbol 0Therm_Enclosure:TYPE-604-T3
- added USB2: U-USBAS04P-F000, 0Library:USB-A-TH_U-A-24DD-Y-2, symbol 0Therm_Enclosure:U-USBAS04P-F000
- J50, J51, J52, J60: footprint Connector_JST:JST_PH_B2B-PH-K_1x02_P2.00mm_Vertical -> Connector_PinSocket_2.54mm:PinSocket_1x02_P2.54mm_Vertical
Connections:
- net +5V: now also DC1.4, J67.1 (Pin_1), J68.1 (Pin_1), USB1.A9 (VBUS), USB1.B9 (VBUS), USB2.1 (VCC)
- net GND: now also DC1.1, DC1.2, DC1.3, DC1.6, H30.1, H31.1, H32.1, H33.1, H34.1, H35.1, H36.1, H37.1, H38.1, H39.1, H40.1, H41.1, J67.2 (Pin_2), J68.2 (Pin_2), USB1.7 (EH), USB1.8 (EH), USB1.A12 (GND), USB1.B12 (GND), USB2.4 (GND), USB2.5, USB2.6
- no-connect marks 0 -> 4
Other:
- note added: "12x 2mm Diode Boards (4 each stack + 2)"
- note added: "Power 5V 30W Rating"
- note removed: "8x 2mm Diode Boards (5 each stack)"

Commit message: Removed files unrelated
Parts:
- J14, J15, J55, J57, J58, J59: LCSC C124418 -> C2897370
Changed lines of the file:
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@@
       (effects (font (size 1.27 1.27)) hide)
     )
-    (property "LCSC" "C124418" (id 4) (at 196.977 47.879 0)
+    (property "LCSC" "C2897370" (id 4) (at 196.977 47.879 0)
       (effects (font (size 1.27 1.27)) hide)
     )
@@
       (effects (font (size 1.27 1.27)) hide)
     )
-    (property "LCSC" "C124418" (id 4) (at 191.897 47.879 0)
+    (property "LCSC" "C2897370" (id 4) (at 191.897 47.879 0)
       (effects (font (size 1.27 1.27)) hide)
     )
@@
       (effects (font (size 1.27 1.27)) hide)
     )
-    (property "LCSC" "C124418" (id 4) (at 74.295 48.895 0)
+    (property "LCSC" "C2897370" (id 4) (at 74.295 48.895 0)
       (effects (font (size 1.27 1.27)) hide)
     )
@@
       (effects (font (size 1.27 1.27)) hide)
     )
-    (property "LCSC" "C124418" (id 4) (at 192.405 121.285 0)
+    (property "LCSC" "C2897370" (id 4) (at 192.405 121.285 0)
       (effects (font (size 1.27 1.27)) hide)
     )
@@
       (effects (font (size 1.27 1.27)) hide)
     )
-    (property "LCSC" "C124418" (id 4) (at 79.375 48.895 0)
+    (property "LCSC" "C2897370" (id 4) (at 79.375 48.895 0)
       (effects (font (size 1.27 1.27)) hide)
     )
@@
       (effects (font (size 1.27 1.27)) hide)
     )
-    (property "LCSC" "C124418" (id 4) (at 187.325 121.285 0)
+    (property "LCSC" "C2897370" (id 4) (at 187.325 121.285 0)
       (effects (font (size 1.27 1.27)) hide)
     )
@@
     )
     (path "/1177b381-35f4-4300-ae70-b7e5fb7ae7dc/7f3ae4e3-f0eb-4b26-bf37-bc74d157a221"
-      (reference "J1") (unit 1) (value "HDMI_A_1.4") (footprint "0Library:HDMI-TH_HDMI-019A")
+      (reference "J1") (unit 1) (value "HDMI_A_1.4") (footprint "0Library:HDMI-TH_HYC12-HDMIA19-61")
     )
     (path "/1177b381-35f4-4300-ae70-b7e5fb7ae7dc/9a8a14b1-05f5-4aaa-aa60-0a085b1fa134"
-      (reference "J2") (unit 1) (value "HDMI_A_1.4") (footprint "0Library:HDMI-TH_HDMI-019A")
+      (reference "J2") (unit 1) (value "HDMI_A_1.4") (footprint "0Library:HDMI-TH_HYC12-HDMIA19-61")
     )
     (path "/1177b381-35f4-4300-ae70-b7e5fb7ae7dc/33eb0e30-6e8a-473f-ad47-216a8a439007"
-      (reference "J3") (unit 1) (value "HDMI_A_1.4") (footprint "0Library:HDMI-TH_HDMI-019A")
+      (reference "J3") (unit 1) (value "HDMI_A_1.4") (footprint "0Library:HDMI-TH_HYC12-HDMIA19-61")
     )
     (path "/1177b381-35f4-4300-ae70-b7e5fb7ae7dc/9b659bc8-59ea-46ce-9f16-63022b7f8b29"
-      (reference "J4") (unit 1) (value "HDMI_A_1.4") (footprint "0Library:HDMI-TH_HDMI-019A")
+      (reference "J4") (unit 1) (value "HDMI_A_1.4") (footprint "0Library:HDMI-TH_HYC12-HDMIA19-61")
     )
     (path "/1177b381-35f4-4300-ae70-b7e5fb7ae7dc/fccd994b-ad06-4c54-a67b-7ca6d3784203"
-      (reference "J5") (unit 1) (value "HDMI_A_1.4") (footprint "0Library:HDMI-TH_HDMI-019A")
+      (reference "J5") (unit 1) (value "HDMI_A_1.4") (footprint "0Library:HDMI-TH_HYC12-HDMIA19-61")
     )
     (path "/1177b381-35f4-4300-ae70-b7e5fb7ae7dc/759fe5fd-eda2-4bb3-aac6-ed0cea27f3f5"
-      (reference "J6") (unit 1) (value "HDMI_A_1.4") (footprint "0Library:HDMI-TH_HDMI-019A")
+      (reference "J6") (unit 1) (value "HDMI_A_1.4") (footprint "0Library:HDMI-TH_HYC12-HDMIA19-61")
     )
     (path "/1177b381-35f4-4300-ae70-b7e5fb7ae7dc/a344ddad-17c4-4704-88db-532a6a8d328c"
-      (reference "J7") (unit 1) (value "HDMI_A_1.4") (footprint "0Library:HDMI-TH_HDMI-019A")
+      (reference "J7") (unit 1) (value "HDMI_A_1.4") (footprint "0Library:HDMI-TH_HYC12-HDMIA19-61")
     )
     (path "/1177b381-35f4-4300-ae70-b7e5fb7ae7dc/98c44a44-830c-4240-81b4-61d3a9378ac2"
-      (reference "J8") (unit 1) (value "HDMI_A_1.4") (footprint "0Library:HDMI-TH_HDMI-019A")
+      (reference "J8") (unit 1) (value "HDMI_A_1.4") (footprint "0Library:HDMI-TH_HYC12-HDMIA19-61")
     )
     (path "/1177b381-35f4-4300-ae70-b7e5fb7ae7dc/af4deb43-05dd-4f0b-a5ad-45ae07fdf40c"
-      (reference "J9") (unit 1) (value "HDMI_A_1.4") (footprint "0Library:HDMI-TH_HDMI-019A")
+      (reference "J9") (unit 1) (value "HDMI_A_1.4") (footprint "0Library:HDMI-TH_HYC12-HDMIA19-61")
     )
     (path "/c0c186eb-9fce-4130-ae7b-b5cd8fe51419"
