File: Motherboard V2/25V_to5V.kicad_sch.kicad_sch (KiCad schematic)
At the start: 13 parts, among them J50 Conn_01x01, J51 Conn_01x01, U2 TDK30-24S05W

Commit message: update
Parts:
- C12: LCSC C5162365 -> C7471899
- L3: LCSC C439009 -> C917352
Changed lines of the file:
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@@
 			)
 		)
-		(property "LCSC" "C439009"
+		(property "LCSC" "C917352"
 			(at 128.905 71.755 90)
 			(effects
@@
 			)
 		)
-		(property "LCSC" "C5162365"
+		(property "LCSC" "C7471899 "
 			(at 97.79 78.105 0)
 			(effects
