File: Motherboard V2/dd-50.kicad_sch (KiCad schematic)
At the start: 40 parts, among them J1 HDMI_A_1.4, J19 JST_SH_Conn_01x04_D HEad, J2 HDMI_A_1.4, J20 JST_SH_Conn_01x04_3Head B, J21 JST_SH_Conn_01x04_3Head A, J22 JST_SH_Conn_01x04_Still, J23 JST_SH_Conn_01x04_4Head B, J24 JST_SH_Conn_01x04_4Head A, J25 JST_SH_Conn_01x04_4Pump Diode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, J26 JST_SH_Conn_01x04_4Pump Diode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, J27 JST_SH_Conn_01x04_3Pump Diode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, J28 JST_SH_Conn_01x04_3Pump Diode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, J29 JST_SH_Conn_01x04_Condenser, J3 HDMI_A_1.4, J30 JST_SH_Conn_01x04_4Switch Dio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, J31 JST_SH_Conn_01x04_4Switch Dio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, J32 Conn_01x02_Still Heater, J33 JST_SH_Conn_01x04_3Switch Dio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, J34 JST_SH_Conn_01x04_3Switch Dio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, J35 Conn_01x02_15 pin Extra, J36 Conn_01x02_4SwitchHeater B, J37 Conn_01x02_4SwitchHeater A, J38 Conn_01x02_3SwitchHeater B, J39 Conn_01x02_3SwitchHeater A, J4 HDMI_A_1.4, J40 JST_SH_Conn_01x04_40K Diode, J41 Conn_01x02_4PumpHeater B, J42 Conn_01x02_4PumpHeater A, J43 JST_SH_Conn_01x04_4K Diode, J44 Conn_01x02_3PumpHeater B, J45 Conn_01x02_3PumpHeater A, J46 Conn_01x02_Extra B, J47 Conn_01x02_Extra A, J48 Conn_01x02_Extra B, J49 Conn_01x02_Extra A, J5 HDMI_A_1.4, J6 HDMI_A_1.4, J7 HDMI_A_1.4, J8 HDMI_A_1.4, J9 HDMI_A_1.4

Commit message: update
Parts:
- removed J46, J48: Conn_01x02_Extra B, Connector_JST:JST_PH_B2B-PH-K_1x02_P2.00mm_Vertical, symbol Connector_Generic:Conn_01x02
- removed J47, J49: Conn_01x02_Extra A, Connector_JST:JST_PH_B2B-PH-K_1x02_P2.00mm_Vertical, symbol Connector_Generic:Conn_01x02
- added J14, J46: JST_SH_Conn_01x04_Extra, Connector_JST:JST_SH_BM04B-SRSS-TB_1x04-1MP_P1.00mm_Vertical, symbol 0JLC:JST_SH_Conn_01x04_i2c_horizontal
Connections:
- net at J6.7 (D0+): now also J46.2 (VCC)
- net at J6.9 (D0-): now also J46.3 (SDA)
- net at J3.7 (D0+): now also J14.2 (VCC)
- net at J3.9 (D0-): now also J14.3 (SDA)
- net at J3.10 (CK+): now also J14.1 (gnd)
- net at J3.12 (CK-): now also J14.4 (SCL)
- net at J6.10 (CK+): now also J46.1 (gnd)
- net at J6.12 (CK-): now also J46.4 (SCL)
